Commit message: Create SFD model

File: models/test_door_6_backup.urdf.xacro (robot description, xacro)
@@ -11,7 +11,5 @@
       <origin rpy="0 0 0" xyz="0 0 0"/>
       <mass value="1000000.0"/>
-      <inertia ixx="0.013102127690" 	ixy="-0.000000514790"	ixz="0.000000965200"
-					iyy="0.017339000240" 	iyz="-0.000017996010"
-								izz="0.004334337460"/>
+      <inertia ixx="0.048966669" ixy="0" ixz="0" iyy="0.046466667" iyz="0" izz="0.0041666669"/>
     </inertial>
     <visual>
@@ -35,7 +33,5 @@
       <origin rpy="0 0 0" xyz="0 0 0"/>
       <mass value="50.0"/>
-      <inertia ixx="0.030386862790" 	ixy="0.000000000330"	ixz="-0.000000216760"
-					iyy="0.035534743650" 	iyz="-0.000000000060"
-								izz="0.005184277950"/>
+      <inertia ixx="0.048966669" ixy="0" ixz="0" iyy="0.046466667" iyz="0" izz="0.0041666669"/>
     </inertial>
     <visual>
@@ -67,7 +63,5 @@
       <origin rpy="0 0 0" xyz="0 0 0"/>
       <mass value="5.0"/>
-      <inertia ixx="0.0000005040778809"	ixy="0.0000000194018051"	ixz="-0.0000000003676693"
-					iyy="0.0000005395705566"	iyz="0.0000000001548617"
-									izz="0.0000004894420410"/>
+      <inertia ixx="0.048966669" ixy="0" ixz="0" iyy="0.046466667" iyz="0" izz="0.0041666669"/>
     </inertial>
     <visual>
@@ -102,5 +96,5 @@
   </gazebo>
  <gazebo reference="door">
-    <self_collide>1</self_collide>
+    <self_collide>0</self_collide>
   </gazebo>
 </robot>

File: models/test_door_7.urdf.xacro (robot description, xacro)
@@ -10,5 +10,5 @@
     <inertial>
       <origin rpy="0 0 0" xyz="0 0 0"/>
-      <mass value="1000000.0"/>
+      <mass value="100.0"/>
       <inertia ixx="0.013102127690" 	ixy="-0.000000514790"	ixz="0.000000965200"
 					iyy="0.017339000240" 	iyz="-0.000017996010"
@@ -34,5 +34,5 @@
     <inertial>
       <origin rpy="0 0 0" xyz="0 0 0"/>
-      <mass value="50.0"/>
+      <mass value="0.1"/>
       <inertia ixx="0.030386862790" 	ixy="0.000000000330"	ixz="-0.000000216760"
 					iyy="0.035534743650" 	iyz="-0.000000000060"
@@ -58,5 +58,5 @@
     <parent link="frame"/>
     <child link="door"/>
-    <dynamics damping="1.0" friction="0.0001"/>
+    <dynamics damping="0.2" friction="0.000001"/>
     <origin xyz="0 0 0"/>
     <axis xyz="0 0 1"/>
@@ -67,7 +67,5 @@
       <origin rpy="0 0 0" xyz="0 0 0"/>
       <mass value="5.0"/>
-      <inertia ixx="0.0000005040778809"	ixy="0.0000000194018051"	ixz="-0.0000000003676693"
-					iyy="0.0000005395705566"	iyz="0.0000000001548617"
-									izz="0.0000004894420410"/>
+      <inertia ixx="0.01" ixy="0" ixz="0" iyy="0.01" iyz="0" izz="0.01"/>
     </inertial>
     <visual>
@@ -90,5 +88,5 @@
     <parent link="door"/>
     <child link="lever"/>
-	<dynamics damping="1.0" friction="0.0001"/>
+	<dynamics damping="0.5" friction="0.000001"/>
     <origin rpy="1.5708 0 0" xyz="-0.79604 -0.06 1.0"/>
 		<axis xyz="0 0 1"/>

File: models/test_door_8.urdf.xacro (robot description, xacro)
@@ -10,5 +10,5 @@
     <inertial>
       <origin rpy="0 0 0" xyz="0 0 0"/>
-      <mass value="1000000.0"/>
+      <mass value="100.0"/>
       <inertia ixx="0.013102127690" 	ixy="-0.000000514790"	ixz="0.000000965200"
 					iyy="0.017339000240" 	iyz="-0.000017996010"
@@ -31,8 +31,11 @@
      </collision>
    </link>
+  <gazebo reference="frame">
+    <material>Gazebo/WoodPallet</material>
+  </gazebo>
    <link name="door">
     <inertial>
       <origin rpy="0 0 0" xyz="0 0 0"/>
-      <mass value="50.0"/>
+      <mass value="0.1"/>
       <inertia ixx="0.030386862790" 	ixy="0.000000000330"	ixz="-0.000000216760"
 					iyy="0.035534743650" 	iyz="-0.000000000060"
@@ -44,7 +47,4 @@
          <mesh filename="package://reemc_door/models/meshes/door4.stl"/>
        </geometry>
-	   <material name="doormat0">
-      <color rgba="0.8 0.8 0.3 1" />
-      </material>
 	  </visual>
      <collision>
@@ -55,8 +55,11 @@
      </collision>
    </link>
+  <gazebo reference="door">
+    <material>Gazebo/Wood</material>
+  </gazebo>
   <joint name="joint_frame_door" type="revolute">
     <parent link="frame"/>
     <child link="door"/>
-    <dynamics damping="1.0" friction="0.0001"/>
+    <dynamics damping="0.2" friction="0.000001"/>
     <origin xyz="0 0 0"/>
     <axis xyz="0 0 1"/>
@@ -67,7 +70,5 @@
       <origin rpy="0 0 0" xyz="0 0 0"/>
       <mass value="5.0"/>
-      <inertia ixx="0.0000005040778809"	ixy="0.0000000194018051"	ixz="-0.0000000003676693"
-					iyy="0.0000005395705566"	iyz="0.0000000001548617"
-									izz="0.0000004894420410"/>
+      <inertia ixx="0.01" ixy="0" ixz="0" iyy="0.01" iyz="0" izz="0.01"/>
     </inertial>
     <visual>
@@ -87,8 +88,11 @@
      </collision>
    </link>
+  <gazebo reference="lever">
+    <material>Gazebo/Gold</material>
+  </gazebo>
    <joint name="joint_door_lever" type="revolute">
     <parent link="door"/>
     <child link="lever"/>
-	<dynamics damping="1.0" friction="0.0001"/>
+	<dynamics damping="0.5" friction="0.000001"/>
     <origin rpy="1.5708 0 0" xyz="-0.79604 -0.06 1.0"/>
 		<axis xyz="0 0 1"/>

File: models/test_door_9.urdf.xacro (robot description, xacro)
@@ -5,10 +5,10 @@
     <parent link="world"/>
     <child link="frame"/>
-    <origin rpy= "0 0 1.571" xyz="0 0 0"/>
+    <origin rpy= "0 0 0" xyz="0 0 0"/>
   </joint>
 <link name="frame">
     <inertial>
       <origin rpy="0 0 0" xyz="0 0 0"/>
-      <mass value="1000000.0"/>
+      <mass value="100.0"/>
       <inertia ixx="0.013102127690" 	ixy="-0.000000514790"	ixz="0.000000965200"
 					iyy="0.017339000240" 	iyz="-0.000017996010"
@@ -31,8 +31,11 @@
      </collision>
    </link>
+  <gazebo reference="frame">
+    <material>Gazebo/WoodPallet</material>
+  </gazebo>
    <link name="door">
     <inertial>
       <origin rpy="0 0 0" xyz="0 0 0"/>
-      <mass value="50.0"/>
+      <mass value="0.1"/>
       <inertia ixx="0.030386862790" 	ixy="0.000000000330"	ixz="-0.000000216760"
 					iyy="0.035534743650" 	iyz="-0.000000000060"
@@ -44,7 +47,4 @@
          <mesh filename="package://reemc_door/models/meshes/door4.stl"/>
        </geometry>
-	   <material name="doormat0">
-      <color rgba="0.8 0.8 0.3 1" />
-      </material>
 	  </visual>
      <collision>
@@ -55,8 +55,11 @@
      </collision>
    </link>
+  <gazebo reference="door">
+    <material>Gazebo/Wood</material>
+  </gazebo>
   <joint name="joint_frame_door" type="revolute">
     <parent link="frame"/>
     <child link="door"/>
-    <dynamics damping="1.0" friction="0.0001"/>
+    <dynamics damping="0.2" friction="0.000001"/>
     <origin xyz="0 0 0"/>
     <axis xyz="0 0 1"/>
@@ -67,7 +70,5 @@
       <origin rpy="0 0 0" xyz="0 0 0"/>
       <mass value="5.0"/>
-      <inertia ixx="0.0000005040778809"	ixy="0.0000000194018051"	ixz="-0.0000000003676693"
-					iyy="0.0000005395705566"	iyz="0.0000000001548617"
-									izz="0.0000004894420410"/>
+      <inertia ixx="0.01" ixy="0" ixz="0" iyy="0.01" iyz="0" izz="0.01"/>
     </inertial>
     <visual>
@@ -87,11 +88,20 @@
      </collision>
    </link>
+  <gazebo reference="lever">
+    <material>Gazebo/Gold</material>
+  </gazebo>
    <joint name="joint_door_lever" type="revolute">
     <parent link="door"/>
     <child link="lever"/>
-	<dynamics damping="1.0" friction="0.0001"/>
+	<!--dynamics damping="0.5" friction="0.000001"/-->
     <origin rpy="1.5708 0 0" xyz="-0.79604 -0.06 1.0"/>
 		<axis xyz="0 0 1"/>
    <limit effort="1000.0" lower="-0.5236" upper="0.0" velocity="0.5"/>
+  <gazebo reference="joint_door_lever">
+    <implicitSpringDamper>true</implicitSpringDamper>
+    <spring_stiffness>10000</spring_stiffness>
+    <spring_reference>0.0</spring_reference>
+    <damping>10.0</damping>
+  </gazebo>
   </joint>
   <gazebo reference="lever">
